File: Controller/Clank_controller/Clank_controller.kicad_sch (KiCad schematic)
At the start: 0 parts

Commit message: udated by FZ
Parts:
- added J? (x7): Limit switch, symbol Connector:Conn_01x02_Male
- added J? (x3): OpticalEnd, symbol Connector:Conn_01x03_Male
- added J?: +5V Conn, symbol Connector:Conn_01x02_Male
- added J?: Extension Connector, symbol Connector_Generic:Conn_02x10_Counter_Clockwise
Connections:
- new net +5V: J?.1 (Pin_1)
- new net GND: J?.2 (Pin_2)
