File: Controller/Clank_controller/Clank_controller.kicad_sch (KiCad schematic)
At the start: 12 parts

Commit message: udated by FZ
Parts:
- added J? (x7): Limit switch, symbol Connector:Conn_01x02_Male
Connections:
- net at J?.1 (Pin_1): now also J?.1 (Pin_1) (x7)
- net at J?.2 (Pin_2): now also J?.2 (Pin_2) (x7)
Other:
- moved on the sheet: J?

Commit message: udated by FZ
Parts:
- removed J? (x14): Limit switch, symbol Connector:Conn_01x02_Male
- removed J? (x3): OpticalEnd, symbol Connector:Conn_01x03_Male
- removed J?: +5V Conn, symbol Connector:Conn_01x02_Male
- removed J?: Extension Connector, symbol Connector_Generic:Conn_02x10_Counter_Clockwise
- added C1: 10uF, Capacitor_THT:CP_Radial_D5.0mm_P2.50mm, symbol Device:C_Polarized_Small
- added C2: 220uF, Capacitor_THT:CP_Radial_D14.0mm_P5.00mm, symbol Device:C_Polarized_Small
- added D1, D2: LED, LED_SMD:LED_1206_3216Metric_Pad1.42x1.75mm_HandSolder, symbol Device:LED
- added H1, H2, H3, H4, H5, H6: M3, MountingHole:MountingHole_3.2mm_M3, symbol Mechanical:MountingHole
- added J1, J2, J3, J4, J5, J6: Limit_SW, Connector_PinHeader_2.54mm:PinHeader_2x02_P2.54mm_Vertical, symbol Connector_Generic:Conn_02x02_Counter_Clockwise
- added J10, J11, J13: Screw_Terminal_01x02, TerminalBlock_MetzConnect:TerminalBlock_MetzConnect_Type011_RT05502HBWC_1x02_P5.00mm_Horizontal, symbol Connector:Screw_Terminal_01x02
- added J12, J14, J15, J17, J18: +5V Conn, Connector_PinHeader_2.54mm:PinHeader_1x02_P2.54mm_Vertical, symbol Connector:Conn_01x02_Male
- added J16: Conn_02x13_Odd_Even, Connector_IDC:IDC-Header_2x13_P2.54mm_Vertical, symbol Connector_Generic:Conn_02x13_Odd_Even
- added J7, J8, J9: Conn_02x03_Counter_Clockwise, Connector_PinHeader_2.54mm:PinHeader_2x03_P2.54mm_Vertical, symbol Connector_Generic:Conn_02x03_Counter_Clockwise
- added R1: 1K, Resistor_SMD:R_1206_3216Metric_Pad1.30x1.75mm_HandSolder, symbol Device:R_Small
- added R2, R3: 10K, Resistor_SMD:R_1206_3216Metric_Pad1.30x1.75mm_HandSolder, symbol Device:R_Small
Connections:
- net +5V: now also C1.1, J10.2 (Pin_2), J12.1 (Pin_1), J7.1 (Pin_1), J7.2 (Pin_2), J8.1 (Pin_1), J8.2 (Pin_2), J9.1 (Pin_1), J9.2 (Pin_2), R1.1
- net GND: now also C1.2, C2.2, D1.1 (K), D2.1 (K), J10.1 (Pin_1), J11.1 (Pin_1), J12.2 (Pin_2), J13.1 (Pin_1), J16.17 (Pin_17), J16.18 (Pin_18), J16.19 (Pin_19), J16.20 (Pin_20), J16.21 (Pin_21), J16.22 (Pin_22), J16.23 (Pin_23), J16.24 (Pin_24), J16.25 (Pin_25), J16.26 (Pin_26), J7.3 (Pin_3), J7.4 (Pin_4), J8.3 (Pin_3), J8.4 (Pin_4), J9.3 (Pin_3), J9.4 (Pin_4), R3.1
- new net: J6.1 (Pin_1), J6.2 (Pin_2)
- new net: J6.3 (Pin_3), J6.4 (Pin_4)
- new net: D2.2 (A), R2.2
- new net: J16.10 (Pin_10), J17.2 (Pin_2)
- new net: J14.2 (Pin_2), J16.11 (Pin_11)
- new net: J16.12 (Pin_12), J17.1 (Pin_1)
- new net: J14.1 (Pin_1), J16.9 (Pin_9)
- new net: J1.1 (Pin_1), J1.2 (Pin_2)
- new net: J1.3 (Pin_3), J1.4 (Pin_4)
- new net: D1.2 (A), R1.2
- new net: J4.1 (Pin_1), J4.2 (Pin_2)
- new net: J4.3 (Pin_3), J4.4 (Pin_4)
- new net: J2.1 (Pin_1), J2.2 (Pin_2)
- new net: J2.3 (Pin_3), J2.4 (Pin_4)
- new net: J3.1 (Pin_1), J3.2 (Pin_2)
- new net: J3.3 (Pin_3), J3.4 (Pin_4)
- new net: J5.1 (Pin_1), J5.2 (Pin_2)
- new net: J5.3 (Pin_3), J5.4 (Pin_4)
- new net +24V: C2.1, J11.2 (Pin_2), J13.2 (Pin_2), J16.1 (Pin_1), J16.2 (Pin_2), J16.3 (Pin_3), J16.4 (Pin_4), J16.5 (Pin_5), J16.6 (Pin_6), J16.7 (Pin_7), J16.8 (Pin_8), R2.1, R3.2
- new net IO_1: J15.1 (Pin_1), J16.13 (Pin_13)
- new net IO_2: J15.2 (Pin_2), J16.15 (Pin_15)
- new net IO_3: J16.14 (Pin_14), J18.2 (Pin_2)
- new net IO_4: J16.16 (Pin_16), J18.1 (Pin_1)
- new net SIG1: J7.5 (Pin_5), J7.6 (Pin_6)
- new net SIG2: J8.5 (Pin_5), J8.6 (Pin_6)
- new net SIG3: J9.5 (Pin_5), J9.6 (Pin_6)
Other:
- note added: "Clank machine Grbl controller extension board."
- note added: "Extension connector"
- note added: "Limit switches"
- note added: "Optical EndStop"
- note added: "Power supply"
