File: Controller/Clank_controller/Clank_controller.kicad_pcb (KiCad board)
At the start: 2 copper layers, 104 x 95 mm, 31 parts, among them J1 Limit_SW, J10 Screw_Terminal_01x02, J11 Screw_Terminal_01x02, J12 +5V Conn, J13 Screw_Terminal_01x02, J14 +5V Conn, J15 +5V Conn, J16 Conn_02x13_Odd_Even, J17 +5V Conn, J18 +5V Conn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

Commit message: udated by FZ
Parts:
- moved J11 50.8 mm to (175.4, 63.0)
- moved J13 50.8 mm to (194.9, 76.8)
- moved J14 50.8 mm to (149.8, 70.8)
- moved J15 50.8 mm to (142.9, 70.8)
- moved J17 50.8 mm to (147.3, 74.5)
- moved R1 50.8 mm to (109.8, 60.7)
- moved D1 50.8 mm to (107.3, 60.8)
- moved H2 50.8 mm to (99.8, 148.2)
- moved H3 50.8 mm to (99.8, 61.2)
- moved H4 50.8 mm to (120.8, 148.2)
- moved H5 50.8 mm to (120.8, 96.2)
- moved J10 50.8 mm to (119.8, 62.8)
- moved J12 50.8 mm to (117.0, 75.7)
- moved C1 50.8 mm to (111.9, 75.8)
- moved C2 50.8 mm to (176.3, 81.2)
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
Commit message: udated by FZ
Routing:
- net +24V: track 12.8 -> 9.01 mm
Changed lines of the file:
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@@
   (segment (start 100.555 94.29) (end 103.095 94.29) (width 0.762) (layer "F.Cu") (net 12))
   (segment (start 100.555 84.45875) (end 103.095 84.45875) (width 0.762) (layer "F.Cu") (net 13))
-  (segment (start 170.41 61.67) (end 170.41 63) (width 0.762) (layer "F.Cu") (net 14))
-  (segment (start 180.83 59.2225) (end 172.8575 59.2225) (width 0.762) (layer "F.Cu") (net 14))
-  (segment (start 172.8575 59.2225) (end 170.41 61.67) (width 0.762) (layer "F.Cu") (net 14))
+  (segment (start 172.7775 59.2225) (end 172.1 59.9) (width 0.508) (layer "F.Cu") (net 14))
+  (segment (start 180.83 59.2225) (end 172.7775 59.2225) (width 0.508) (layer "F.Cu") (net 14))
   (via (at 164.83 74.75) (size 0.762) (drill 0.381) (layers "F.Cu" "B.Cu") (free) (net 14))
   (via (at 192.33 67.25) (size 0.762) (drill 0.381) (layers "F.Cu" "B.Cu") (free) (net 14))
@@
   )
   (zone (net 2) (net_name "GND") (layer "F.Cu") (hatch edge 0.508)
-    (connect_pads yes (clearance 0.254))
+    (connect_pads (clearance 0.254))
     (min_thickness 0.254) (filled_areas_thickness no)
     (fill yes (thermal_gap 0.254) (thermal_bridge_width 0.508))
@@
     (connect_pads (clearance 0.254))
     (min_thickness 0.254) (filled_areas_thickness no)
-    (fill yes (thermal_gap 0.508) (thermal_bridge_width 0.508))
+    (fill yes (thermal_gap 0.254) (thermal_bridge_width 0.508))
     (polygon
       (pts
@@
   (zone (net 1) (net_name "+5V") (layer "F.Cu") (hatch edge 0.508)
     (priority 1)
-    (connect_pads yes (clearance 0.254))
-    (min_thickness 0.254) (filled_areas_thickness no)
-    (fill yes (thermal_gap 0.508) (thermal_bridge_width 0.508))
+    (connect_pads (clearance 0.254))
+    (min_thickness 0.254) (filled_areas_thickness no)
+    (fill yes (thermal_gap 0.254) (thermal_bridge_width 0.508))
     (polygon
       (pts
@@
   (zone (net 14) (net_name "+24V") (layer "F.Cu") (hatch edge 0.508)
     (priority 2)
-    (connect_pads yes (clearance 0.254))
+    (connect_pads (clearance 0.254))
     (min_thickness 0.254) (filled_areas_thickness no)
     (fill yes (thermal_gap 0.254) (thermal_bridge_width 0.508))
@@
   (zone (net 14) (net_name "+24V") (layer "B.Cu") (hatch edge 0.508)
     (priority 1)
-    (connect_pads yes (clearance 0.254))
+    (connect_pads (clearance 0.254))
     (min_thickness 0.254) (filled_areas_thickness no)
     (fill yes (thermal_gap 0.254) (thermal_bridge_width 0.508))
@@
   )
   (zone (net 2) (net_name "GND") (layer "B.Cu") (hatch edge 0.508)
-    (connect_pads yes (clearance 0.254))
-    (min_thickness 0.254) (filled_areas_thickness no)
-    (fill yes (thermal_gap 0.254) (thermal_bridge_width 0.508))
+    (connect_pads (clearance 0.254))
+    (min_thickness 0.254) (filled_areas_thickness no)
+    (fill yes (thermal_gap 0.254) (thermal_bridge_width 0.508))
