File: Modules/Spindle_Driver/Spindle_Driver.kicad_pcb (KiCad board)
At the start: 2 copper layers, 66.7 x 83 mm, 24 parts, among them J1 PWR in, J3 Ctrl in, J4 To Spindle, J5 +5V Conn, J6 +5V Conn, J7 +5V Conn, J8 Conn_02x13_Odd_Even, J9 +5V Conn, Q1 IRF540N

Commit message: udated by FZ
Routing:
- net /PWM: track 50.1 -> 49.0 mm
- net GND: track 5.87 -> 5.79 mm, vias 3 -> 4
Other:
- board text added: "+24V"
- board text added: "Clank machine - Spindle Driver module"
- board text added: "Fangzheng Liu fzliu@mit.edu"
- board text added: "Motor+"
- board text added: "Motor-"
- board text added: "PWM"
Changed lines of the file:
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@@
     )
   )
+  (gr_line (start 140 130) (end 145.25 130) (layer "F.SilkS") (width 1.5))
+  (gr_line (start 140 127.25) (end 145.25 127.25) (layer "F.SilkS") (width 1.5))
+  (gr_line (start 137.25 124.75) (end 137.25 132.75) (layer "F.SilkS") (width 1.5))
+  (gr_line (start 140 132.75) (end 145.25 132.75) (layer "F.SilkS") (width 1.5))
+  (gr_line (start 140 132.75) (end 140 127.25) (layer "F.SilkS") (width 1.5))
+  (gr_line (start 137.25 124.75) (end 145.25 124.75) (layer "F.SilkS") (width 1.5))
   (gr_line (start 168 142) (end 133.3 142) (layer "Edge.Cuts") (width 0.1))
   (gr_line (start 133.3 142) (end 133.3 67) (layer "Edge.Cuts") (width 0.1))
@@
   (gr_line (start 200 67) (end 200 150) (layer "Edge.Cuts") (width 0.1))
   (gr_line (start 200 150) (end 168 150) (layer "Edge.Cuts") (width 0.1))
+  (gr_text "PWM" (at 146.75 91.5 90) (layer "F.SilkS")
+    (effects (font (size 1 1) (thickness 0.15)))
+  )
+  (gr_text "Clank machine\n- Spindle Driver module" (at 147.25 131.5) (layer "F.SilkS")
+    (effects (font (size 1.5 1.5) (thickness 0.2)) (justify left))
+  )
+  (gr_text "+24V" (at 184.75 80.75) (layer "F.SilkS")
+    (effects (font (size 1 1) (thickness 0.15)))
+  )
+  (gr_text "Fangzheng Liu\nfzliu@mit.edu" (at 136.375 137.25) (layer "F.SilkS")
+    (effects (font (size 1.2 1.2) (thickness 0.1)) (justify left))
+  )
+  (gr_text "Motor+" (at 146.5 109 90) (layer "F.SilkS")
+    (effects (font (size 1 1) (thickness 0.15)))
+  )
+  (gr_text "Motor-" (at 146.5 114.75 90) (layer "F.SilkS")
+    (effects (font (size 1 1) (thickness 0.15)))
+  )
   (segment (start 184.825 72.675) (end 184.825 72.8) (width 0.508) (layer "F.Cu") (net 1))
   (segment (start 186.5875 70.9125) (end 184.825 72.675) (width 0.508) (layer "F.Cu") (net 1))
@@
   (via (at 166 100) (size 0.8) (drill 0.4) (layers "F.Cu" "B.Cu") (free) (net 1))
   (via (at 166 98) (size 0.8) (drill 0.4) (layers "F.Cu" "B.Cu") (free) (net 1))
-  (segment (start 163.2 112.8625) (end 161.6 114.4625) (width 0.508) (layer "F.Cu") (net 2))
-  (segment (start 161.6 117.93) (end 161.59 117.94) (width 0.508) (layer "F.Cu") (net 2))
-  (segment (start 161.6 114.4625) (end 161.6 117.93) (width 0.508) (layer "F.Cu") (net 2))
-  (segment (start 163.2 112.7375) (end 163.2 112.8625) (width 0.508) (layer "F.Cu") (net 2))
+  (segment (start 163.2 112.7375) (end 164.9075 112.7375) (width 0.762) (layer "F.Cu") (net 2))
+  (segment (start 161.6 114.4625) (end 161.6 116.26) (width 0.762) (layer "F.Cu") (net 2))
+  (segment (start 164.9075 112.7375) (end 166.52 114.35) (width 0.762) (layer "F.Cu") (net 2))
+  (via (at 161.6 116.26) (size 0.8) (drill 0.4) (layers "F.Cu" "B.Cu") (net 2))
   (via (at 151.32 96.42) (size 0.8) (drill 0.4) (layers "F.Cu" "B.Cu") (net 2))
-  (via (at 161.59 117.94) (size 0.8) (drill 0.4) (layers "F.Cu" "B.Cu") (net 2))
   (via (at 191.72 70.86) (size 0.8) (drill 0.4) (layers "F.Cu" "B.Cu") (net 2))
+  (via (at 166.52 114.35) (size 0.8) (drill 0.4) (layers "F.Cu" "B.Cu") (net 2))
   (segment (start 158.3025 101.41) (end 158.3 101.4125) (width 0.762) (layer "F.Cu") (net 4))
   (segment (start 159.91 101.41) (end 158.3025 101.41) (width 0.762) (layer "F.Cu") (net 4))
@@
   (segment (start 147.8975 91.4) (end 149.4875 92.99) (width 0.254) (layer "F.Cu") (net 6))
   (segment (start 138.425 91.4) (end 147.8975 91.4) (width 0.254) (layer "F.Cu") (net 6))
-  (segment (start 150.3725 70.06) (end 138.17 70.06) (width 0.254) (layer "B.Cu") (net 6))
-  (segment (start 135.735 72.495) (end 135.735 81.11) (width 0.254) (layer "B.Cu") (net 6))
-  (segment (start 152.26 71.9475) (end 150.3725 70.06) (width 0.254) (layer "B.Cu") (net 6))
+  (segment (start 151.26 77.73) (end 136.34 77.73) (width 0.254) (layer "B.Cu") (net 6))
+  (segment (start 153.569489 73.256989) (end 153.569489 75.420511) (width 0.254) (layer "B.Cu") (net 6))
+  (segment (start 136.34 77.73) (end 135.735 78.335) (width 0.254) (layer "B.Cu") (net 6))
+  (segment (start 135.735 78.335) (end 135.735 81.11) (width 0.254) (layer "B.Cu") (net 6))
   (segment (start 135.735 81.11) (end 136.955511 82.330511) (width 0.254) (layer "B.Cu") (net 6))
-  (segment (start 138.17 70.06) (end 135.735 72.495) (width 0.254) (layer "B.Cu") (net 6))
+  (segment (start 152.26 71.9475) (end 153.569489 73.256989) (width 0.254) (layer "B.Cu") (net 6))
+  (segment (start 153.569489 75.420511) (end 151.26 77.73) (width 0.254) (layer "B.Cu") (net 6))
   (segment (start 136.955511 82.330511) (end 136.955511 89.930511) (width 0.254) (layer "B.Cu") (net 6))
   (segment (start 136.955511 89.930511) (end 138.425 91.4) (width 0.254) (layer "B.Cu") (net 6))
@@
         (xy 136.4 108.6)
         (xy 137 108)
-        (xy 151.4 108)
       )
     )
@@
   )
   (zone (net 2) (net_name "GND") (layer "B.Cu") (hatch edge 0.508)
-    (connect_pads (clearance 0.508))
-    (min_thickness 0.508) (filled_areas_thickness no)
+    (connect_pads (clearance 0.254))
+    (min_thickness 0.254) (filled_areas_thickness no)
     (fill yes (thermal_gap 0.254) (thermal_bridge_width 0.508))
     (polygon
       (pts
-        (xy 201 151)
-        (xy 167 151)
-        (xy 167 143)
-        (xy 133 143)
+        (xy 200.5 150.25)
+        (xy 167.75 150.25)
+        (xy 167.75 142.25)
+        (xy 133 142.25)
         (xy 133 66)
-        (xy 201 66)
+        (xy 200.5 66)
       )
     )
@@
         (xy 173.5 102)
         (xy 171.5 104)
-        (xy 171.5 109)
-        (xy 164 116.5)
-        (xy 160 116.5)
-        (xy 159 115.5)
-        (xy 159 114.5)
-        (xy 160.5 113)
-        (xy 163.5 113)
-        (xy 167 109.5)
+        (xy 171.5 107.5)
+        (xy 164 115)
+        (xy 159.75 115)
+        (xy 159 114.25)
+        (xy 159 112.25)
+        (xy 159.75 111.5)
+        (xy 163.5 111.5)
+        (xy 167 108)
         (xy 167 104)
         (xy 165.5 102.5)

Commit message: udated by FZ
Parts:
- moved C2 1.70 mm to (163.2, 115.3), turned to -90 degrees
- moved C4 1.70 mm to (161.6, 115.3)
- moved C1 1.60 mm to (163.5, 88.1)
Routing:
- net GND: track 5.79 -> 0.00 mm
- net /Motor-: track 0.00 -> 3.83 mm
Changed lines of the file:
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@@
   )
   (footprint "Capacitor_THT:CP_Radial_D14.0mm_P5.00mm" (layer "F.Cu")
-    (at 163.5 86.5 180)
+    (at 163.5 88.1 180)
     (descr "CP, Radial series, Radial, pin pitch=5.00mm, , diameter=14mm, Electrolytic Capacitor")
     (tags "CP Radial series Radial pin pitch 5.00mm  diameter 14mm Electrolytic Capacitor")
@@
   )
   (footprint "Capacitor_SMD:C_0603_1608Metric_Pad1.08x0.95mm_HandSolder" (layer "F.Cu")
-    (at 161.6 113.6 -90)
+    (at 161.6 115.3 -90)
     (descr "Capacitor SMD 0603 (1608 Metric), square (rectangular) end terminal, IPC_7351 nominal with elongated pad for handsoldering. (Body size source: IPC-SM-782 page 76, https://www.pcb-3d.com/wordpress/wp-content/uploads/ipc-sm-782a_amendment_1_and_2.pdf), generated with kicad-footprint-generator")
     (tags "capacitor handsolder")
@@
   )
   (footprint "Capacitor_SMD:C_0603_1608Metric_Pad1.08x0.95mm_HandSolder" (layer "F.Cu")
-    (at 163.2 113.6 90)
+    (at 163.2 115.3 -90)
     (descr "Capacitor SMD 0603 (1608 Metric), square (rectangular) end terminal, IPC_7351 nominal with elongated pad for handsoldering. (Body size source: IPC-SM-782 page 76, https://www.pcb-3d.com/wordpress/wp-content/uploads/ipc-sm-782a_amendment_1_and_2.pdf), generated with kicad-footprint-generator")
     (tags "capacitor handsolder")
@@
     (fp_line (start 0.8 0.4) (end -0.8 0.4) (layer "F.Fab") (width 0.1))
     (fp_line (start 0.8 -0.4) (end 0.8 0.4) (layer "F.Fab") (width 0.1))
-    (pad "1" smd roundrect (at -0.8625 0 90) (size 1.075 0.95) (layers "F.Cu" "F.Paste" "F.Mask") (roundrect_rratio 0.25)
+    (pad "1" smd roundrect (at -0.8625 0 270) (size 1.075 0.95) (layers "F.Cu" "F.Paste" "F.Mask") (roundrect_rratio 0.25)
       (net 1 "+24V") (pintype "passive"))
-    (pad "2" smd roundrect (at 0.8625 0 90) (size 1.075 0.95) (layers "F.Cu" "F.Paste" "F.Mask") (roundrect_rratio 0.25)
+    (pad "2" smd roundrect (at 0.8625 0 270) (size 1.075 0.95) (layers "F.Cu" "F.Paste" "F.Mask") (roundrect_rratio 0.25)
       (net 2 "GND") (pintype "passive"))
     (model "${KICAD6_3DMODEL_DIR}/Capacitor_SMD.3dshapes/C_0603_1608Metric.wrl"
@@
   (via (at 166 100) (size 0.8) (drill 0.4) (layers "F.Cu" "B.Cu") (free) (net 1))
   (via (at 166 98) (size 0.8) (drill 0.4) (layers "F.Cu" "B.Cu") (free) (net 1))
-  (segment (start 163.2 112.7375) (end 164.9075 112.7375) (width 0.762) (layer "F.Cu") (net 2))
-  (segment (start 161.6 114.4625) (end 161.6 116.26) (width 0.762) (layer "F.Cu") (net 2))
-  (segment (start 164.9075 112.7375) (end 166.52 114.35) (width 0.762) (layer "F.Cu") (net 2))
-  (via (at 161.6 116.26) (size 0.8) (drill 0.4) (layers "F.Cu" "B.Cu") (net 2))
   (via (at 151.32 96.42) (size 0.8) (drill 0.4) (layers "F.Cu" "B.Cu") (net 2))
+  (via (at 163.2 116.2) (size 0.8) (drill 0.4) (layers "F.Cu" "B.Cu") (net 2))
   (via (at 191.72 70.86) (size 0.8) (drill 0.4) (layers "F.Cu" "B.Cu") (net 2))
-  (via (at 166.52 114.35) (size 0.8) (drill 0.4) (layers "F.Cu" "B.Cu") (net 2))
+  (via (at 161.6 116.2) (size 0.8) (drill 0.4) (layers "F.Cu" "B.Cu") (net 2))
+  (segment (start 161.6 114.291778) (end 160.045722 112.7375) (width 0.762) (layer "F.Cu") (net 3))
+  (segment (start 160.045722 112.7375) (end 160 112.7375) (width 0.762) (layer "F.Cu") (net 3))
+  (segment (start 161.6 114.4375) (end 161.6 113) (width 0.762) (layer "F.Cu") (net 3))
+  (segment (start 161.6 114.4375) (end 161.6 114.291778) (width 0.762) (layer "F.Cu") (net 3))
   (segment (start 158.3025 101.41) (end 158.3 101.4125) (width 0.762) (layer "F.Cu") (net 4))
   (segment (start 159.91 101.41) (end 158.3025 101.41) (width 0.762) (layer "F.Cu") (net 4))
@@
     (connect_pads yes (clearance 0.508))
     (min_thickness 0.508) (filled_areas_thickness no)
-    (fill yes (thermal_gap 0.508) (thermal_bridge_width 0.508))
+    (fill yes (thermal_gap 0.254) (thermal_bridge_width 0.508))
     (polygon
       (pts
@@
         (xy 157.25 100.25)
         (xy 156 101.5)
-        (xy 156 106.5)
-        (xy 151 106.5)
-        (xy 151 99)
-        (xy 161.3 89.3)
-        (xy 161.5 70)
+        (xy 156 106.8)
+        (xy 150.7 106.8)
+        (xy 150.7 98.7)
+        (xy 161.1 89.3)
+        (xy 161.2 70.1)
         (xy 173 70)
         (xy 173 75)
