File: Modules/Spindle_Driver/Spindle_Driver.kicad_sch (KiCad schematic)
At the start: 0 parts

Commit message: udated by FZ
Parts:
- added C1: (no value), symbol Device:C_Polarized_Small
- added C2, C4: 0.1uF, symbol Device:C_Small
- added C3: (no value), symbol Device:C_Small
- added D1: (no value), symbol Diode:1N5822
- added D2: LED, symbol Device:LED
- added D3: (no value), symbol Device:LED
- added H1, H2: (no value), symbol Mechanical:MountingHole
- added J1, J3, J4: (no value), symbol Connector:Screw_Terminal_01x02
- added J5, J6, J7, J9: +5V Conn, Connector_PinHeader_2.54mm:PinHeader_1x02_P2.54mm_Vertical, symbol Connector:Conn_01x02_Male
- added J8: Conn_02x13_Odd_Even, Connector_IDC:IDC-Header_2x13_P2.54mm_Vertical, symbol Connector_Generic:Conn_02x13_Odd_Even
- added L1, L2: (no value), symbol Device:L_Small
- added Q1: (no value), symbol Transistor_FET:IRF540N
- added R1, R4: 10K, symbol Device:R_Small
- added R2, R3: (no value), symbol Device:R_Small
Connections:
- new net: D3.2 (A), R4.1
- new net: J6.1 (Pin_1), J8.12 (Pin_12)
- new net: J6.2 (Pin_2), J8.10 (Pin_10)
- new net: Q1.1 (G), R2.2, R3.2
- new net: D2.2 (A), R1.1
- new net: J7.1 (Pin_1), J8.13 (Pin_13)
- new net: J8.16 (Pin_16), J9.1 (Pin_1)
- new net: J8.14 (Pin_14), J9.2 (Pin_2)
- new net: J5.1 (Pin_1), J8.9 (Pin_9)
- new net: J5.2 (Pin_2), J8.11 (Pin_11)
- new net +24V: C1.1, C2.1, C3.1, D1.1 (K), J1.1 (Pin_1), J8.1 (Pin_1), J8.2 (Pin_2), J8.3 (Pin_3), J8.4 (Pin_4), J8.5 (Pin_5), J8.6 (Pin_6), J8.7 (Pin_7), J8.8 (Pin_8), L1.1, R1.2, R4.2
- new net GND: C1.2, C2.2, C4.2, D3.1 (K), J1.2 (Pin_2), J3.2 (Pin_2), J8.17 (Pin_17), J8.18 (Pin_18), J8.19 (Pin_19), J8.20 (Pin_20), J8.21 (Pin_21), J8.22 (Pin_22), J8.23 (Pin_23), J8.24 (Pin_24), J8.25 (Pin_25), J8.26 (Pin_26), Q1.3 (S), R3.1
- new net Motor+: J4.1 (Pin_1), L1.2
- new net Motor-: C3.2, C4.1, J4.2 (Pin_2), L2.2
- new net PWM: J3.1 (Pin_1), J7.2 (Pin_2), J8.15 (Pin_15), R2.1
- new net net_D: D1.2 (A), D2.1 (K), L2.1, Q1.2 (D)
Other:
- company: (none) -> MIT Media Lab
- title: (none) -> Spindle_Driver_board

Commit message: udated by FZ
Parts:
- C1: value (none) -> 220uF; footprint (none) -> Capacitor_THT:CP_Radial_D14.0mm_P5.00mm
- C2, C4: footprint (none) -> Capacitor_SMD:C_0603_1608Metric_Pad1.08x0.95mm_HandSolder
- C3: value (none) -> 0.1uF; footprint (none) -> Capacitor_SMD:C_0603_1608Metric_Pad1.08x0.95mm_HandSolder
- D1: value (none) -> 1N5822; footprint (none) -> Diode_THT:D_DO-201AD_P15.24mm_Horizontal
- D2: footprint (none) -> LED_SMD:LED_0603_1608Metric_Pad1.05x0.95mm_HandSolder
- D3: value (none) -> LED; footprint (none) -> LED_SMD:LED_0603_1608Metric_Pad1.05x0.95mm_HandSolder
- H1, H2: value (none) -> M3; footprint (none) -> MountingHole:MountingHole_3.2mm_M3
- J1: value (none) -> PWR in; footprint (none) -> TerminalBlock_MetzConnect:TerminalBlock_MetzConnect_Type011_RT05502HBWC_1x02_P5.00mm_Horizontal
- J3: value (none) -> Ctrl in; footprint (none) -> TerminalBlock_MetzConnect:TerminalBlock_MetzConnect_Type011_RT05502HBWC_1x02_P5.00mm_Horizontal
- J4: value (none) -> To Spindle; footprint (none) -> TerminalBlock_MetzConnect:TerminalBlock_MetzConnect_Type011_RT05502HBWC_1x02_P5.00mm_Horizontal
- L1, L2: value (none) -> 3.3uH; footprint (none) -> Mylib:SRP7028A-3R3M
- Q1: value (none) -> IRF540N; footprint (none) -> Package_TO_SOT_THT:TO-220-3_Vertical
- R1, R4: footprint (none) -> Resistor_SMD:R_0603_1608Metric_Pad0.98x0.95mm_HandSolder
- R2: value (none) -> 150; footprint (none) -> Resistor_SMD:R_0603_1608Metric_Pad0.98x0.95mm_HandSolder
- R3: value (none) -> 10K; footprint (none) -> Resistor_SMD:R_0603_1608Metric_Pad0.98x0.95mm_HandSolder
Changed lines of the file:
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@@
       (effects (font (size 1.27 1.27)) (justify left))
     )
-    (property "Value" "" (id 1) (at 88.9 100.7622 0)
-      (effects (font (size 1.27 1.27)) (justify left))
-    )
-    (property "Footprint" "" (id 2) (at 86.36 99.06 0)
+    (property "Value" "M3" (id 1) (at 88.9 100.7622 0)
+      (effects (font (size 1.27 1.27)) (justify left))
+    )
+    (property "Footprint" "MountingHole:MountingHole_3.2mm_M3" (id 2) (at 86.36 99.06 0)
       (effects (font (size 1.27 1.27)) hide)
     )
@@
     (in_bom yes) (on_board yes) (fields_autoplaced)
     (property "Reference" "L2" (id 0) (at 139.7 44.1792 90))
-    (property "Value" "" (id 1) (at 139.7 46.7161 90))
-    (property "Footprint" "" (id 2) (at 139.7 48.26 0)
+    (property "Value" "3.3uH" (id 1) (at 139.7 46.7161 90))
+    (property "Footprint" "Mylib:SRP7028A-3R3M" (id 2) (at 139.7 48.26 0)
       (effects (font (size 1.27 1.27)) hide)
     )
@@
     (in_bom yes) (on_board yes) (fields_autoplaced)
     (property "Reference" "D3" (id 0) (at 42.2275 71.6112 0))
-    (property "Value" "" (id 1) (at 42.2275 74.1481 0))
-    (property "Footprint" "" (id 2) (at 40.64 77.47 0)
+    (property "Value" "LED" (id 1) (at 42.2275 74.1481 0))
+    (property "Footprint" "LED_SMD:LED_0603_1608Metric_Pad1.05x0.95mm_HandSolder" (id 2) (at 40.64 77.47 0)
       (effects (font (size 1.27 1.27)) hide)
     )
@@
       (effects (font (size 1.27 1.27)) (justify left))
     )
-    (property "Value" "" (id 1) (at 82.169 36.7161 0)
-      (effects (font (size 1.27 1.27)) (justify left))
-    )
-    (property "Footprint" "" (id 2) (at 80.01 35.56 0)
+    (property "Value" "220uF" (id 1) (at 82.169 36.7161 0)
+      (effects (font (size 1.27 1.27)) (justify left))
+    )
+    (property "Footprint" "Capacitor_THT:CP_Radial_D14.0mm_P5.00mm" (id 2) (at 80.01 35.56 0)
       (effects (font (size 1.27 1.27)) hide)
     )
@@
       (effects (font (size 1.27 1.27)) (justify left))
     )
-    (property "Footprint" "" (id 2) (at 125.73 38.1 0)
+    (property "Footprint" "Capacitor_SMD:C_0603_1608Metric_Pad1.08x0.95mm_HandSolder" (id 2) (at 125.73 38.1 0)
       (effects (font (size 1.27 1.27)) hide)
     )
@@
     (in_bom yes) (on_board yes) (fields_autoplaced)
     (property "Reference" "L1" (id 0) (at 139.7 26.3992 90))
-    (property "Value" "" (id 1) (at 139.7 28.9361 90))
-    (property "Footprint" "" (id 2) (at 139.7 30.48 0)
+    (property "Value" "3.3uH" (id 1) (at 139.7 28.9361 90))
+    (property "Footprint" "Mylib:SRP7028A-3R3M" (id 2) (at 139.7 30.48 0)
       (effects (font (size 1.27 1.27)) hide)
     )
@@
       (effects (font (size 1.27 1.27)) (justify left))
     )
-    (property "Value" "" (id 1) (at 100.33 100.7622 0)
-      (effects (font (size 1.27 1.27)) (justify left))
-    )
-    (property "Footprint" "" (id 2) (at 97.79 99.06 0)
+    (property "Value" "M3" (id 1) (at 100.33 100.7622 0)
+      (effects (font (size 1.27 1.27)) (justify left))
+    )
+    (property "Footprint" "MountingHole:MountingHole_3.2mm_M3" (id 2) (at 97.79 99.06 0)
       (effects (font (size 1.27 1.27)) hide)
     )
@@
     (in_bom yes) (on_board yes) (fields_autoplaced)
     (property "Reference" "J1" (id 0) (at 41.91 20.4302 0))
-    (property "Value" "" (id 1) (at 41.91 22.9671 0))
-    (property "Footprint" "" (id 2) (at 41.91 25.4 0)
+    (property "Value" "PWR in" (id 1) (at 41.91 22.9671 0))
+    (property "Footprint" "TerminalBlock_MetzConnect:TerminalBlock_MetzConnect_Type011_RT05502HBWC_1x02_P5.00mm_Horizontal" (id 2) (at 41.91 25.4 0)
       (effects (font (size 1.27 1.27)) hide)
     )
@@
     (in_bom yes) (on_board yes) (fields_autoplaced)
     (property "Reference" "R2" (id 0) (at 83.82 50.1736 90))
-    (property "Value" "" (id 1) (at 83.82 52.7105 90))
-    (property "Footprint" "" (id 2) (at 83.82 54.61 0)
+    (property "Value" "150" (id 1) (at 83.82 52.7105 90))
+    (property "Footprint" "Resistor_SMD:R_0603_1608Metric_Pad0.98x0.95mm_HandSolder" (id 2) (at 83.82 54.61 0)
       (effects (font (size 1.27 1.27)) hide)
     )
@@
     (in_bom yes) (on_board yes)
     (property "Reference" "J4" (id 0) (at 171.45 92.71 0))
-    (property "Value" "" (id 1) (at 179.07 96.52 0))
-    (property "Footprint" "" (id 2) (at 171.45 97.79 0)
+    (property "Value" "To Spindle" (id 1) (at 179.07 96.52 0))
+    (property "Footprint" "TerminalBlock_MetzConnect:TerminalBlock_MetzConnect_Type011_RT05502HBWC_1x02_P5.00mm_Horizontal" (id 2) (at 171.45 97.79 0)
       (effects (font (size 1.27 1.27)) hide)
     )
@@
       (effects (font (size 1.27 1.27)) (justify right))
     )
-    (property "Footprint" "" (id 2) (at 99.06 41.91 0)
+    (property "Footprint" "LED_SMD:LED_0603_1608Metric_Pad1.05x0.95mm_HandSolder" (id 2) (at 99.06 41.91 0)
       (effects (font (size 1.27 1.27)) hide)
     )
@@
       (effects (font (size 1.27 1.27)) (justify right))
     )
-    (property "Footprint" "" (id 2) (at 99.06 34.29 0)
+    (property "Footprint" "Resistor_SMD:R_0603_1608Metric_Pad0.98x0.95mm_HandSolder" (id 2) (at 99.06 34.29 0)
       (effects (font (size 1.27 1.27)) hide)
     )
@@
       (effects (font (size 1.27 1.27)) hide)
     )
-    (property "Value" "" (id 1) (at 48.26 20.5542 0))
+    (property "Value" "+24V" (id 1) (at 48.26 20.5542 0))
     (property "Footprint" "" (id 2) (at 48.26 24.13 0)
       (effects (font (size 1.27 1.27)) hide)
@@
       (effects (font (size 1.27 1.27)) hide)
     )
-    (property "Value" "" (id 1) (at 22.86 29.464 0))
+    (property "Value" "PWR_FLAG" (id 1) (at 22.86 29.464 0))
     (property "Footprint" "" (id 2) (at 22.86 25.4 0)
       (effects (font (size 1.27 1.27)) hide)
@@
       (effects (font (size 1.27 1.27)) (justify left))
     )
-    (property "Value" "" (id 1) (at 144.5641 41.0785 0)
-      (effects (font (size 1.27 1.27)) (justify left))
-    )
-    (property "Footprint" "" (id 2) (at 142.24 39.37 0)
+    (property "Value" "0.1uF" (id 1) (at 144.5641 41.0785 0)
+      (effects (font (size 1.27 1.27)) (justify left))
+    )
+    (property "Footprint" "Capacitor_SMD:C_0603_1608Metric_Pad1.08x0.95mm_HandSolder" (id 2) (at 142.24 39.37 0)
       (effects (font (size 1.27 1.27)) hide)
     )
@@
     (in_bom yes) (on_board yes)
     (property "Reference" "J3" (id 0) (at 41.91 39.4802 0))
-    (property "Value" "" (id 1) (at 41.91 42.0171 0))
-    (property "Footprint" "" (id 2) (at 41.91 44.45 0)
+    (property "Value" "Ctrl in" (id 1) (at 41.91 42.0171 0))
+    (property "Footprint" "TerminalBlock_MetzConnect:TerminalBlock_MetzConnect_Type011_RT05502HBWC_1x02_P5.00mm_Horizontal" (id 2) (at 41.91 44.45 0)
       (effects (font (size 1.27 1.27)) hide)
     )
@@
       (effects (font (size 1.27 1.27)) (justify right))
     )
-    (property "Value" "" (id 1) (at 90.3986 61.3922 0)
-      (effects (font (size 1.27 1.27)) (justify right))
-    )
-    (property "Footprint" "" (id 2) (at 88.9 59.69 0)
+    (property "Value" "10K" (id 1) (at 90.3986 61.3922 0)
+      (effects (font (size 1.27 1.27)) (justify right))
+    )
+    (property "Footprint" "Resistor_SMD:R_0603_1608Metric_Pad0.98x0.95mm_HandSolder" (id 2) (at 88.9 59.69 0)
       (effects (font (size 1.27 1.27)) hide)
     )
@@
       (effects (font (size 1.27 1.27)) (justify left))
     )
-    (property "Footprint" "" (id 2) (at 147.32 53.34 0)
+    (property "Footprint" "Capacitor_SMD:C_0603_1608Metric_Pad1.08x0.95mm_HandSolder" (id 2) (at 147.32 53.34 0)
       (effects (font (size 1.27 1.27)) hide)
     )
@@
       (effects (font (size 1.27 1.27)) (justify left))
     )
-    (property "Value" "" (id 1) (at 101.727 56.3122 0)
-      (effects (font (size 1.27 1.27)) (justify left))
-    )
-    (property "Footprint" "" (id 2) (at 102.87 56.515 0)
+    (property "Value" "IRF540N" (id 1) (at 101.727 56.3122 0)
+      (effects (font (size 1.27 1.27)) (justify left))
+    )
+    (property "Footprint" "Package_TO_SOT_THT:TO-220-3_Vertical" (id 2) (at 102.87 56.515 0)
       (effects (font (size 1.27 1.27) italic) (justify left) hide)
     )
@@
       (effects (font (size 1.27 1.27)) (justify left))
     )
-    (property "Value" "" (id 1) (at 113.792 42.0247 90)
-      (effects (font (size 1.27 1.27)) (justify left))
-    )
-    (property "Footprint" "" (id 2) (at 107.315 40.64 0)
+    (property "Value" "1N5822" (id 1) (at 113.792 42.0247 90)
+      (effects (font (size 1.27 1.27)) (justify left))
+    )
+    (property "Footprint" "Diode_THT:D_DO-201AD_P15.24mm_Horizontal" (id 2) (at 107.315 40.64 0)
       (effects (font (size 1.27 1.27)) hide)
     )
@@
       (effects (font (size 1.27 1.27)) hide)
     )
-    (property "Value" "" (id 1) (at 48.26 52.7034 0))
+    (property "Value" "GND" (id 1) (at 48.26 52.7034 0))
     (property "Footprint" "" (id 2) (at 48.26 48.26 0)
       (effects (font (size 1.27 1.27)) hide)
@@
     (property "Reference" "R4" (id 0) (at 31.75 73.0336 90))
     (property "Value" "10K" (id 1) (at 31.75 75.5705 90))
-    (property "Footprint" "" (id 2) (at 31.75 77.47 0)
-      (effects (font (size 1.27 1.27)) hide)
-    )
+    (property "Footprint" "Resistor_SMD:R_0603_1608Metric_Pad0.98x0.95mm_HandSolder" (id 2) (at 31.75 77.47 0)
+      (effects (font (size 1.27 1.27)) hide)
+    )
